Commit message: laser added

File: src/amr-ros-config/description/urdf/pioneer3at.urdf.xacro (robot description, xacro)
@@ -1,18 +1,7 @@
 <?xml version="1.0"?>
-<robot xmlns:sensor="http://playerstage.sourceforge.net/gazebo/xmlschema/#sensor"
-       xmlns:controller="http://playerstage.sourceforge.net/gazebo/xmlschema/#controller"
-       xmlns:interface="http://playerstage.sourceforge.net/gazebo/xmlschema/#interface"
-       xmlns:xacro="http://ros.org/wiki/xacro"
-name="pioneer3at">
+<robot xmlns:xacro="http://ros.org/wiki/xacro" name="pioneer3at">
 <xacro:include filename="$(find amr_robots_description)/urdf/materials.xacro" />
 <!-- Chassis -->
 	<link name="base_link">
-		<!--  For pointers on inertial and gazebo-related parameters see
-		       * http://wiki.ros.org/urdf/Tutorials/Adding%20Physical%20and%20Collision%20Properties%20to%20a%20URDF%20Model
-                       * http://answers.gazebosim.org/question/4372/the-inertia-matrix-explained/
-		       * http://gazebosim.org/tutorials?tut=inertia&cat=build_robot, and
-                       * http://gazebosim.org/tutorials/?tut=ros_urdf
-                       * http://en.wikipedia.org/wiki/List_of_moment_of_inertia_tensors
-                -->
 		<inertial>
 			<mass value="21.5"/> <!-- P3AT 18.6kg plus three batteries @ 2.4kg each  minus four wheels @ 1.4 kg ea and top plate @ 0.1 kg-->
@@ -46,43 +35,43 @@
 		</material>
 	</gazebo>
-  <joint name="imu_joint" type="fixed">
-    <axis xyz="1 0 0"/> <!-- 0 1 0 -->
-    <origin xyz="0 0 0.19"/>
-    <parent link="base_link"/>
-    <child link="imu_link"/>
-  </joint>
-  <joint name="basefootprint_joint" type="fixed">
-    <axis xyz="1 0 0"/> <!-- 0 1 0 -->
-    <origin xyz="0 0 0.19"/>
-    <parent link="base_link"/>
-    <child link="base_footprint"/>
-  </joint>
-<link name="base_footprint">
-  <visual>
-    <origin rpy="0 0 0" xyz="0 0 0"/>
-    <geometry>
-      <box size="0.001 0.001 0.001"/>
-    </geometry>
-  </visual>
-</link>
-<link name="imu_link">
-  <inertial>
-    <mass value="0.001"/>
-    <origin rpy="0 0 0" xyz="0 0 0"/>
-    <inertia ixx="0.0001" ixy="0" ixz="0" iyy="0.000001" iyz="0" izz="0.0001"/>
-  </inertial>
-  <visual>
-    <origin rpy="0 0 0" xyz="0 0 0"/>
-    <geometry>
-      <box size="0.001 0.001 0.001"/>
-    </geometry>
-  </visual>
-  <collision>
-    <origin rpy="0 0 0" xyz="0 0 0"/>
-    <geometry>
-      <box size=".001 .001 .001"/>
-    </geometry>
-  </collision>
-</link>
+	<joint name="imu_joint" type="fixed">
+		<axis xyz="1 0 0"/> <!-- 0 1 0 -->
+		<origin xyz="0 0 0.19"/>
+	    	<parent link="base_link"/>
+	    	<child link="imu_link"/>
+	</joint>
+	<joint name="basefootprint_joint" type="fixed">
+	    	<axis xyz="1 0 0"/> <!-- 0 1 0 -->
+	    	<origin xyz="0 0 0.19"/>
+	    	<parent link="base_link"/>
+	    	<child link="base_footprint"/>
+	</joint>
+	<link name="base_footprint">
+		<visual>
+	    		<origin rpy="0 0 0" xyz="0 0 0"/>
+	   		<geometry>
+	      		<box size="0.001 0.001 0.001"/>
+	   		</geometry>
+	  	</visual>
+	</link>
+	<link name="imu_link">
+	  	<inertial>
+		    	<mass value="0.001"/>
+		    	<origin rpy="0 0 0" xyz="0 0 0"/>
+		    	<inertia ixx="0.0001" ixy="0" ixz="0" iyy="0.000001" iyz="0" izz="0.0001"/>
+	 	</inertial>
+	  	<visual>
+	    		<origin rpy="0 0 0" xyz="0 0 0"/>
+	    		<geometry>
+	      			<box size="0.001 0.001 0.001"/>
+	    		</geometry>
+	 	</visual>
+	  	<collision>
+	    		<origin rpy="0 0 0" xyz="0 0 0"/>
+	    		<geometry>
+	      			<box size=".001 .001 .001"/>
+	    		</geometry>
+	  	</collision>
+		</link>
 <!-- Top -->
 	<link name="top_plate">
@@ -196,4 +185,30 @@
 		<child link="back_sonar"/>
 	</joint>
+	<joint name="hokuyo_joint" type="fixed">
+		<axis xyz="0 1 0" />
+		<origin xyz="0 0 0.31" rpy="0 0 0"/>
+		<parent link="base_link"/>
+		<child link="hokuyo_link"/>
+	</joint>
+	<!-- Hokuyo Laser -->
+	<link name="hokuyo_link">
+		<collision>
+			<origin xyz="0 0 0" rpy="0 0 0"/>
+	      		<geometry>
+	    			<box size="0.1 0.1 0.1"/>
+	      		</geometry>
+	    	</collision>
+		<visual>
+			<origin xyz="0 0 0" rpy="0 0 0"/>
+		      	<geometry>
+				<mesh filename="package://amr_robots_description/meshes/p3at_meshes/hokuyo.dae"/>
+		      	</geometry>
+		</visual>
+		<inertial>
+	      		<mass value="1e-5" />
+	      		<origin xyz="0 0 0" rpy="0 0 0"/>
+	      		<inertia ixx="1e-6" ixy="0" ixz="0" iyy="1e-6" iyz="0" izz="1e-6" />
+	    	</inertial>
+	  </link>
 <xacro:macro name="p3at_drive_side" params="side reflect">
   <!-- Front Axles + Wheels + Hubcaps -->
@@ -457,4 +472,40 @@
   </gazebo>
 </xacro:macro>
+<!-- hokuyo -->
+  <gazebo reference="hokuyo_link">
+    <sensor type="gpu_ray" name="head_hokuyo_sensor">
+      <pose>3 3 3 1 1 1</pose>
+      <visualize>true</visualize>
+      <update_rate>40</update_rate>
+      <ray>
+        <scan>
+          <horizontal>
+            <samples>720</samples>
+            <resolution>1</resolution>
+            <min_angle>-1.570796</min_angle>
+            <max_angle>1.570796</max_angle>
+          </horizontal>
+        </scan>
+        <range>
+          <min>0.10</min>
+          <max>4.0</max>
+          <resolution>0.01</resolution>
+        </range>
+        <noise>
+          <type>gaussian</type>
+          <!-- Noise parameters based on published spec for Hokuyo laser
+               achieving "+-30mm" accuracy at range < 10m.  A mean of 0.0m and
+               stddev of 0.01m will put 99.7% of samples within 0.03m of the true
+               reading. -->
+          <mean>0.0</mean>
+          <stddev>0.01</stddev>
+        </noise>
+      </ray>
+      <plugin name="gazebo_ros_head_hokuyo_controller" filename="libgazebo_ros_gpu_laser.so">
+        <topicName>laserScan</topicName>
+        <frameName>hokuyo_link</frameName>
+      </plugin>
+    </sensor>
+  </gazebo>
 <xacro:macro name="p3at_gazebo_ext">
 <gazebo>

Commit message: sensor performance optimazation and bug fix

File: src/amr-ros-config/description/urdf/pioneer3at.urdf.xacro (robot description, xacro)
@@ -211,4 +211,12 @@
 	    	</inertial>
 	  </link>
+	<link name="hokuyo_scanLink">
+	</link>
+	<joint name="hokuyo_scanJoint" type="fixed">
+		<axis xyz="0 1 0" />
+		<origin xyz="0 0 0.03" rpy="0 0 0"/>
+		<parent link="hokuyo_link"/>
+		<child link="hokuyo_scanLink"/>
+	</joint>
 <xacro:macro name="p3at_drive_side" params="side reflect">
   <!-- Front Axles + Wheels + Hubcaps -->
@@ -473,7 +481,7 @@
 </xacro:macro>
 <!-- hokuyo -->
-  <gazebo reference="hokuyo_link">
-    <sensor type="gpu_ray" name="head_hokuyo_sensor">
-      <pose>3 3 3 1 1 1</pose>
+  <gazebo reference="hokuyo_scanLink">
+    <sensor type="ray" name="head_hokuyo_sensor">
+      <pose>0.0 0.0 0.0 0.0 0.0 0.0</pose>
       <visualize>true</visualize>
       <update_rate>40</update_rate>
@@ -502,7 +510,7 @@
         </noise>
       </ray>
-      <plugin name="gazebo_ros_head_hokuyo_controller" filename="libgazebo_ros_gpu_laser.so">
+      <plugin name="gazebo_ros_head_hokuyo_controller" filename="libgazebo_ros_laser.so">
         <topicName>laserScan</topicName>
-        <frameName>hokuyo_link</frameName>
+        <frameName>hokuyo_scanLink</frameName>
       </plugin>
     </sensor>

Commit message: frame finished

File: src/amr-ros-config/description/urdf/pioneer3at.urdf.xacro (robot description, xacro)
@@ -447,35 +447,4 @@
   <!-- see http://gazebosim.org/tutorials/?tut=ros_urdf -->
   <gazebo reference="p3at_back_${side}_wheel">
-    <kp>1000000.0</kp> <!-- kp and kd for rubber -->
-    <kd>100.0</kd>
-    <mu1>1.0</mu1> <!-- was 10 -->
-    <mu2>1.0</mu2>
-      <!-- how to get these into <surface><friction><ode>... ?
-        slip1 0.5 /slip1
-         slip2 0 /slip2
-      -->
-    <fdir1>0 1 0</fdir1> <!-- is this correct? -->
-    <maxVel>1.0</maxVel>
-    <minDepth>0.00</minDepth>
-    <material>
-          		<ambient>1 0 0 0</ambient>
-          		<diffuse>1 0 0 0</diffuse>
-          		<specular>0 0 0 1</specular>
-          		<emissive>0 0 0 1</emissive>
-		</material>
-  </gazebo>
-  <gazebo reference="p3at_front_${side}_wheel">
-    <kp>1000000.0</kp> <!-- kp and kd for rubber -->
-    <kd>100.0</kd>
-    <mu1>1.0</mu1> <!-- was 10 -->
-    <mu2>1.0</mu2>
-      <!-- how to get these into <surface><friction><ode>... ?
-        slip1 0.5 /slip1
-         slip2 0 /slip2
-      -->
-    <fdir1>0 1 0</fdir1> <!-- is this correct? -->
-    <maxVel>1.0</maxVel>
-    <minDepth>0.00</minDepth>
-    <material value="Gazebo/Black" />
   </gazebo>
 </xacro:macro>
@@ -490,5 +459,5 @@
           <horizontal>
             <samples>720</samples>
-            <resolution>1</resolution>
+            <!--<resolution>1</resolution>-->
             <min_angle>-1.570796</min_angle>
             <max_angle>1.570796</max_angle>
